Commit message: Upload LND geometric collision meshes

File: urdf/common/instruments/roll/roll_4670.urdf.xacro (robot description, xacro)
@@ -21,5 +21,5 @@
         <origin rpy="-${PI_2} 0.0 0.0" xyz="0.0 0.0 0.02975"/>
         <geometry>
-          <mesh filename="package://dvrk_model/meshes/instruments/roll/4670/roll_4670_collision.obj" scale="0.1 0.1 0.1"/>
+          <mesh filename="package://dvrk_model/meshes/instruments/roll/4670/roll_4670_collision_geometric.obj" scale="0.1 0.1 0.1"/>
         </geometry>
       </collision>

File: urdf/common/instruments/tip/tip_006.urdf.xacro (robot description, xacro)
@@ -34,5 +34,5 @@
         <origin rpy="0.0 0.0 0.0" xyz="0.0 0.0 0.0"/>
         <geometry>
-          <mesh filename="package://dvrk_model/meshes/instruments/tip/006/tip_006_1_collision.obj"/>
+          <mesh filename="package://dvrk_model/meshes/instruments/tip/006/tip_006_1_collision_geometric.obj"/>
         </geometry>
       </collision>
@@ -56,5 +56,5 @@
         <origin rpy="0.0 0.0 0.0" xyz="0.0 0.0 0.0"/>
         <geometry>
-          <mesh filename="package://dvrk_model/meshes/instruments/tip/006/tip_006_2_collision.obj"/>
+          <mesh filename="package://dvrk_model/meshes/instruments/tip/006/tip_006_2_collision_geometric.obj"/>
         </geometry>
       </collision>

File: urdf/common/instruments/wrist_pitch/wrist_pitch_0091.urdf.xacro (robot description, xacro)
@@ -20,5 +20,5 @@
         <origin rpy="0.0 ${PI_2} ${PI_2}" xyz="0.0295 0.0 0.0"/>
         <geometry>
-          <mesh filename="package://dvrk_model/meshes/instruments/wrist_pitch/0091/wrist_pitch_0091_collision.obj" scale="0.1 0.1 0.1"/>
+          <mesh filename="package://dvrk_model/meshes/instruments/wrist_pitch/0091/wrist_pitch_0091_collision_geometric.STL" scale="0.1 0.1 0.1"/>
         </geometry>
       </collision>

Commit message: updated convex meshes

File: urdf/common/instruments/roll/roll_4670.urdf.xacro (robot description, xacro)
@@ -19,8 +19,9 @@
       </visual>
       <collision>
-        <origin rpy="-${PI_2} 0.0 0.0" xyz="0.0 0.0 0.02975"/>
+        <origin rpy="0.0 0.0 0.0" xyz="0.0 0.0 0.33627975"/>
         <geometry>
-          <mesh filename="package://dvrk_model/meshes/instruments/roll/4670/roll_4670_collision_geometric.obj" scale="0.1 0.1 0.1"/>
+          <cylinder radius="0.0043725" length="0.5596247"/>
         </geometry>
+        <material name="collision_red"><color rgba="1.0 0.0 0.0 1.0"/></material>
       </collision>
     </link>

File: urdf/common/instruments/tip/tip_006.urdf.xacro (robot description, xacro)
@@ -31,9 +31,73 @@
         </geometry>
       </visual>
-      <collision>
+      <collision name="jaw_1_collision_00">
         <origin rpy="0.0 0.0 0.0" xyz="0.0 0.0 0.0"/>
         <geometry>
-          <mesh filename="package://dvrk_model/meshes/instruments/tip/006/tip_006_1_collision_geometric.obj"/>
+          <mesh filename="package://dvrk_model/meshes/instruments/tip/006/collision_hulls/tip_006_1_convex_hull_00.obj"/>
         </geometry>
+        <material name="collision_red"><color rgba="1.0 0.0 0.0 1.0"/></material>
+      </collision>
+      <collision name="jaw_1_collision_01">
+        <origin rpy="0.0 0.0 0.0" xyz="0.0 0.0 0.0"/>
+        <geometry>
+          <mesh filename="package://dvrk_model/meshes/instruments/tip/006/collision_hulls/tip_006_1_convex_hull_01.obj"/>
+        </geometry>
+        <material name="collision_red"><color rgba="1.0 0.0 0.0 1.0"/></material>
+      </collision>
+      <collision name="jaw_1_collision_02">
+        <origin rpy="0.0 0.0 0.0" xyz="0.0 0.0 0.0"/>
+        <geometry>
+          <mesh filename="package://dvrk_model/meshes/instruments/tip/006/collision_hulls/tip_006_1_convex_hull_02.obj"/>
+        </geometry>
+        <material name="collision_red"><color rgba="1.0 0.0 0.0 1.0"/></material>
+      </collision>
+      <collision name="jaw_1_collision_03">
+        <origin rpy="0.0 0.0 0.0" xyz="0.0 0.0 0.0"/>
+        <geometry>
+          <mesh filename="package://dvrk_model/meshes/instruments/tip/006/collision_hulls/tip_006_1_convex_hull_03.obj"/>
+        </geometry>
+        <material name="collision_red"><color rgba="1.0 0.0 0.0 1.0"/></material>
+      </collision>
+      <collision name="jaw_1_collision_04">
+        <origin rpy="0.0 0.0 0.0" xyz="0.0 0.0 0.0"/>
+        <geometry>
+          <mesh filename="package://dvrk_model/meshes/instruments/tip/006/collision_hulls/tip_006_1_convex_hull_04.obj"/>
+        </geometry>
+        <material name="collision_red"><color rgba="1.0 0.0 0.0 1.0"/></material>
+      </collision>
+      <collision name="jaw_1_collision_05">
+        <origin rpy="0.0 0.0 0.0" xyz="0.0 0.0 0.0"/>
+        <geometry>
+          <mesh filename="package://dvrk_model/meshes/instruments/tip/006/collision_hulls/tip_006_1_convex_hull_05.obj"/>
+        </geometry>
+        <material name="collision_red"><color rgba="1.0 0.0 0.0 1.0"/></material>
+      </collision>
+      <collision name="jaw_1_collision_06">
+        <origin rpy="0.0 0.0 0.0" xyz="0.0 0.0 0.0"/>
+        <geometry>
+          <mesh filename="package://dvrk_model/meshes/instruments/tip/006/collision_hulls/tip_006_1_convex_hull_06.obj"/>
+        </geometry>
+        <material name="collision_red"><color rgba="1.0 0.0 0.0 1.0"/></material>
+      </collision>
+      <collision name="jaw_1_collision_07">
+        <origin rpy="0.0 0.0 0.0" xyz="0.0 0.0 0.0"/>
+        <geometry>
+          <mesh filename="package://dvrk_model/meshes/instruments/tip/006/collision_hulls/tip_006_1_convex_hull_07.obj"/>
+        </geometry>
+        <material name="collision_red"><color rgba="1.0 0.0 0.0 1.0"/></material>
+      </collision>
+      <collision name="jaw_1_collision_08">
+        <origin rpy="0.0 0.0 0.0" xyz="0.0 0.0 0.0"/>
+        <geometry>
+          <mesh filename="package://dvrk_model/meshes/instruments/tip/006/collision_hulls/tip_006_1_convex_hull_08.obj"/>
+        </geometry>
+        <material name="collision_red"><color rgba="1.0 0.0 0.0 1.0"/></material>
+      </collision>
+      <collision name="jaw_1_collision_09">
+        <origin rpy="0.0 0.0 0.0" xyz="0.0 0.0 0.0"/>
+        <geometry>
+          <mesh filename="package://dvrk_model/meshes/instruments/tip/006/collision_hulls/tip_006_1_convex_hull_09.obj"/>
+        </geometry>
+        <material name="collision_red"><color rgba="1.0 0.0 0.0 1.0"/></material>
       </collision>
     </link>
@@ -53,9 +117,73 @@
         </geometry>
       </visual>
-      <collision>
+      <collision name="jaw_2_collision_00">
         <origin rpy="0.0 0.0 0.0" xyz="0.0 0.0 0.0"/>
         <geometry>
-          <mesh filename="package://dvrk_model/meshes/instruments/tip/006/tip_006_2_collision_geometric.obj"/>
+          <mesh filename="package://dvrk_model/meshes/instruments/tip/006/collision_hulls/tip_006_2_convex_hull_00.obj"/>
         </geometry>
+        <material name="collision_red"><color rgba="1.0 0.0 0.0 1.0"/></material>
+      </collision>
+      <collision name="jaw_2_collision_01">
+        <origin rpy="0.0 0.0 0.0" xyz="0.0 0.0 0.0"/>
+        <geometry>
+          <mesh filename="package://dvrk_model/meshes/instruments/tip/006/collision_hulls/tip_006_2_convex_hull_01.obj"/>
+        </geometry>
+        <material name="collision_red"><color rgba="1.0 0.0 0.0 1.0"/></material>
+      </collision>
+      <collision name="jaw_2_collision_02">
+        <origin rpy="0.0 0.0 0.0" xyz="0.0 0.0 0.0"/>
+        <geometry>
+          <mesh filename="package://dvrk_model/meshes/instruments/tip/006/collision_hulls/tip_006_2_convex_hull_02.obj"/>
+        </geometry>
+        <material name="collision_red"><color rgba="1.0 0.0 0.0 1.0"/></material>
+      </collision>
+      <collision name="jaw_2_collision_03">
+        <origin rpy="0.0 0.0 0.0" xyz="0.0 0.0 0.0"/>
+        <geometry>
+          <mesh filename="package://dvrk_model/meshes/instruments/tip/006/collision_hulls/tip_006_2_convex_hull_03.obj"/>
+        </geometry>
+        <material name="collision_red"><color rgba="1.0 0.0 0.0 1.0"/></material>
+      </collision>
+      <collision name="jaw_2_collision_04">
+        <origin rpy="0.0 0.0 0.0" xyz="0.0 0.0 0.0"/>
+        <geometry>
+          <mesh filename="package://dvrk_model/meshes/instruments/tip/006/collision_hulls/tip_006_2_convex_hull_04.obj"/>
+        </geometry>
+        <material name="collision_red"><color rgba="1.0 0.0 0.0 1.0"/></material>
+      </collision>
+      <collision name="jaw_2_collision_05">
+        <origin rpy="0.0 0.0 0.0" xyz="0.0 0.0 0.0"/>
+        <geometry>
+          <mesh filename="package://dvrk_model/meshes/instruments/tip/006/collision_hulls/tip_006_2_convex_hull_05.obj"/>
+        </geometry>
+        <material name="collision_red"><color rgba="1.0 0.0 0.0 1.0"/></material>
+      </collision>
+      <collision name="jaw_2_collision_06">
+        <origin rpy="0.0 0.0 0.0" xyz="0.0 0.0 0.0"/>
+        <geometry>
+          <mesh filename="package://dvrk_model/meshes/instruments/tip/006/collision_hulls/tip_006_2_convex_hull_06.obj"/>
+        </geometry>
+        <material name="collision_red"><color rgba="1.0 0.0 0.0 1.0"/></material>
+      </collision>
+      <collision name="jaw_2_collision_07">
+        <origin rpy="0.0 0.0 0.0" xyz="0.0 0.0 0.0"/>
+        <geometry>
+          <mesh filename="package://dvrk_model/meshes/instruments/tip/006/collision_hulls/tip_006_2_convex_hull_07.obj"/>
+        </geometry>
+        <material name="collision_red"><color rgba="1.0 0.0 0.0 1.0"/></material>
+      </collision>
+      <collision name="jaw_2_collision_08">
+        <origin rpy="0.0 0.0 0.0" xyz="0.0 0.0 0.0"/>
+        <geometry>
+          <mesh filename="package://dvrk_model/meshes/instruments/tip/006/collision_hulls/tip_006_2_convex_hull_08.obj"/>
+        </geometry>
+        <material name="collision_red"><color rgba="1.0 0.0 0.0 1.0"/></material>
+      </collision>
+      <collision name="jaw_2_collision_09">
+        <origin rpy="0.0 0.0 0.0" xyz="0.0 0.0 0.0"/>
+        <geometry>
+          <mesh filename="package://dvrk_model/meshes/instruments/tip/006/collision_hulls/tip_006_2_convex_hull_09.obj"/>
+        </geometry>
+        <material name="collision_red"><color rgba="1.0 0.0 0.0 1.0"/></material>
       </collision>
     </link>

File: urdf/common/instruments/wrist_pitch/wrist_pitch_0091.urdf.xacro (robot description, xacro)
@@ -17,9 +17,87 @@
         </geometry>
       </visual>
-      <collision>
+      <collision name="wrist_pitch_collision_00">
         <origin rpy="0.0 ${PI_2} ${PI_2}" xyz="0.0295 0.0 0.0"/>
         <geometry>
-          <mesh filename="package://dvrk_model/meshes/instruments/wrist_pitch/0091/wrist_pitch_0091_collision_geometric.STL" scale="0.1 0.1 0.1"/>
+          <mesh filename="package://dvrk_model/meshes/instruments/wrist_pitch/0091/collision_hulls/wrist_pitch_0091_convex_hull_00.obj" scale="0.1 0.1 0.1"/>
         </geometry>
+        <material name="collision_red"><color rgba="1.0 0.0 0.0 1.0"/></material>
+      </collision>
+      <collision name="wrist_pitch_collision_01">
+        <origin rpy="0.0 ${PI_2} ${PI_2}" xyz="0.0295 0.0 0.0"/>
+        <geometry>
+          <mesh filename="package://dvrk_model/meshes/instruments/wrist_pitch/0091/collision_hulls/wrist_pitch_0091_convex_hull_01.obj" scale="0.1 0.1 0.1"/>
+        </geometry>
+        <material name="collision_red"><color rgba="1.0 0.0 0.0 1.0"/></material>
+      </collision>
+      <collision name="wrist_pitch_collision_02">
+        <origin rpy="0.0 ${PI_2} ${PI_2}" xyz="0.0295 0.0 0.0"/>
+        <geometry>
+          <mesh filename="package://dvrk_model/meshes/instruments/wrist_pitch/0091/collision_hulls/wrist_pitch_0091_convex_hull_02.obj" scale="0.1 0.1 0.1"/>
+        </geometry>
+        <material name="collision_red"><color rgba="1.0 0.0 0.0 1.0"/></material>
+      </collision>
+      <collision name="wrist_pitch_collision_03">
+        <origin rpy="0.0 ${PI_2} ${PI_2}" xyz="0.0295 0.0 0.0"/>
+        <geometry>
+          <mesh filename="package://dvrk_model/meshes/instruments/wrist_pitch/0091/collision_hulls/wrist_pitch_0091_convex_hull_03.obj" scale="0.1 0.1 0.1"/>
+        </geometry>
+        <material name="collision_red"><color rgba="1.0 0.0 0.0 1.0"/></material>
+      </collision>
+      <collision name="wrist_pitch_collision_04">
+        <origin rpy="0.0 ${PI_2} ${PI_2}" xyz="0.0295 0.0 0.0"/>
+        <geometry>
+          <mesh filename="package://dvrk_model/meshes/instruments/wrist_pitch/0091/collision_hulls/wrist_pitch_0091_convex_hull_04.obj" scale="0.1 0.1 0.1"/>
+        </geometry>
+        <material name="collision_red"><color rgba="1.0 0.0 0.0 1.0"/></material>
+      </collision>
+      <collision name="wrist_pitch_collision_05">
+        <origin rpy="0.0 ${PI_2} ${PI_2}" xyz="0.0295 0.0 0.0"/>
+        <geometry>
+          <mesh filename="package://dvrk_model/meshes/instruments/wrist_pitch/0091/collision_hulls/wrist_pitch_0091_convex_hull_05.obj" scale="0.1 0.1 0.1"/>
+        </geometry>
+        <material name="collision_red"><color rgba="1.0 0.0 0.0 1.0"/></material>
+      </collision>
+      <collision name="wrist_pitch_collision_06">
+        <origin rpy="0.0 ${PI_2} ${PI_2}" xyz="0.0295 0.0 0.0"/>
+        <geometry>
+          <mesh filename="package://dvrk_model/meshes/instruments/wrist_pitch/0091/collision_hulls/wrist_pitch_0091_convex_hull_06.obj" scale="0.1 0.1 0.1"/>
+        </geometry>
+        <material name="collision_red"><color rgba="1.0 0.0 0.0 1.0"/></material>
+      </collision>
+      <collision name="wrist_pitch_collision_07">
+        <origin rpy="0.0 ${PI_2} ${PI_2}" xyz="0.0295 0.0 0.0"/>
+        <geometry>
+          <mesh filename="package://dvrk_model/meshes/instruments/wrist_pitch/0091/collision_hulls/wrist_pitch_0091_convex_hull_07.obj" scale="0.1 0.1 0.1"/>
+        </geometry>
+        <material name="collision_red"><color rgba="1.0 0.0 0.0 1.0"/></material>
+      </collision>
+      <collision name="wrist_pitch_collision_08">
+        <origin rpy="0.0 ${PI_2} ${PI_2}" xyz="0.0295 0.0 0.0"/>
+        <geometry>
+          <mesh filename="package://dvrk_model/meshes/instruments/wrist_pitch/0091/collision_hulls/wrist_pitch_0091_convex_hull_08.obj" scale="0.1 0.1 0.1"/>
+        </geometry>
+        <material name="collision_red"><color rgba="1.0 0.0 0.0 1.0"/></material>
+      </collision>
+      <collision name="wrist_pitch_collision_09">
+        <origin rpy="0.0 ${PI_2} ${PI_2}" xyz="0.0295 0.0 0.0"/>
+        <geometry>
+          <mesh filename="package://dvrk_model/meshes/instruments/wrist_pitch/0091/collision_hulls/wrist_pitch_0091_convex_hull_09.obj" scale="0.1 0.1 0.1"/>
+        </geometry>
+        <material name="collision_red"><color rgba="1.0 0.0 0.0 1.0"/></material>
+      </collision>
+      <collision name="wrist_pitch_collision_10">
+        <origin rpy="0.0 ${PI_2} ${PI_2}" xyz="0.0295 0.0 0.0"/>
+        <geometry>
+          <mesh filename="package://dvrk_model/meshes/instruments/wrist_pitch/0091/collision_hulls/wrist_pitch_0091_convex_hull_10.obj" scale="0.1 0.1 0.1"/>
+        </geometry>
+        <material name="collision_red"><color rgba="1.0 0.0 0.0 1.0"/></material>
+      </collision>
+      <collision name="wrist_pitch_collision_11">
+        <origin rpy="0.0 ${PI_2} ${PI_2}" xyz="0.0295 0.0 0.0"/>
+        <geometry>
+          <mesh filename="package://dvrk_model/meshes/instruments/wrist_pitch/0091/collision_hulls/wrist_pitch_0091_convex_hull_11.obj" scale="0.1 0.1 0.1"/>
+        </geometry>
+        <material name="collision_red"><color rgba="1.0 0.0 0.0 1.0"/></material>
       </collision>
     </link>

File: urdf/common/instruments/wrist_yaw/wrist_yaw_0091.urdf.xacro (robot description, xacro)
@@ -20,6 +20,7 @@
         <origin rpy="0.0 0.0 0.0" xyz="0.0 0.0 -0.000236"/>
         <geometry>
-          <cylinder radius="0.005" length="0.010"/>
+          <mesh filename="package://dvrk_model/meshes/instruments/wrist_yaw/0091/wrist_yaw_0091_collision_geometric.obj"/>
         </geometry>
+        <material name="collision_red"><color rgba="1.0 0.0 0.0 1.0"/></material>
       </collision>
     </link>
