Commit message: updated roll mesh for lnd

File: urdf/common/instruments/roll/roll_4162.urdf.xacro (robot description, xacro)
@@ -18,9 +18,10 @@
         <material name="roll_4670_shaft"><color rgba="0.55 0.55 0.55 1"/></material>
       </visual>
-      <collision>
-        <origin rpy="-${PI_2} 0.0 0.0" xyz="0.0 0.0 0.02975"/>
+      <collision name="roll_collision">
+        <origin rpy="-${PI_2} 0.0 ${PI_2}" xyz="0.0 0.0 0.02975"/>
         <geometry>
-          <mesh filename="package://dvrk_model/meshes/instruments/roll/4670/roll_4670.obj" scale="0.1 0.1 0.1"/>
+          <mesh filename="package://dvrk_model/meshes/instruments/roll/4670/roll_4670_collision_convex_cylinder.obj" scale="0.1 0.1 0.1"/>
         </geometry>
+        <material name="collision_red"><color rgba="1.0 0.0 0.0 1.0"/></material>
       </collision>
     </link>

File: urdf/common/instruments/roll/roll_4670.urdf.xacro (robot description, xacro)
@@ -18,8 +18,8 @@
         <material name="roll_4670_shaft"><color rgba="0.55 0.55 0.55 1"/></material>
       </visual>
-      <collision>
-        <origin rpy="0.0 0.0 0.0" xyz="0.0 0.0 0.33627975"/>
+      <collision name="roll_collision">
+        <origin rpy="-${PI_2} 0.0 ${PI_2}" xyz="0.0 0.0 0.02975"/>
         <geometry>
-          <cylinder radius="0.0043725" length="0.5596247"/>
+          <mesh filename="package://dvrk_model/meshes/instruments/roll/4670/roll_4670_collision_convex_cylinder.obj" scale="0.1 0.1 0.1"/>
         </geometry>
         <material name="collision_red"><color rgba="1.0 0.0 0.0 1.0"/></material>

Commit message: uniform convex hull update for lnd

File: urdf/common/instruments/roll/roll_4162.urdf.xacro (robot description, xacro)
@@ -21,5 +21,5 @@
         <origin rpy="-${PI_2} 0.0 ${PI_2}" xyz="0.0 0.0 0.02975"/>
         <geometry>
-          <mesh filename="package://dvrk_model/meshes/instruments/roll/4670/roll_4670_collision_convex_cylinder.obj" scale="0.1 0.1 0.1"/>
+          <mesh filename="package://dvrk_model/meshes/instruments/roll/4670/collision_hulls/roll_4670_convex_hull_00.obj" scale="0.1 0.1 0.1"/>
         </geometry>
         <material name="collision_red"><color rgba="1.0 0.0 0.0 1.0"/></material>

File: urdf/common/instruments/roll/roll_4670.urdf.xacro (robot description, xacro)
@@ -21,5 +21,5 @@
         <origin rpy="-${PI_2} 0.0 ${PI_2}" xyz="0.0 0.0 0.02975"/>
         <geometry>
-          <mesh filename="package://dvrk_model/meshes/instruments/roll/4670/roll_4670_collision_convex_cylinder.obj" scale="0.1 0.1 0.1"/>
+          <mesh filename="package://dvrk_model/meshes/instruments/roll/4670/collision_hulls/roll_4670_convex_hull_00.obj" scale="0.1 0.1 0.1"/>
         </geometry>
         <material name="collision_red"><color rgba="1.0 0.0 0.0 1.0"/></material>

File: urdf/common/instruments/wrist_yaw/wrist_yaw_0091.urdf.xacro (robot description, xacro)
@@ -17,8 +17,8 @@
         </geometry>
       </visual>
-      <collision>
+      <collision name="wrist_yaw_collision_00">
         <origin rpy="0.0 0.0 0.0" xyz="0.0 0.0 -0.000236"/>
         <geometry>
-          <mesh filename="package://dvrk_model/meshes/instruments/wrist_yaw/0091/wrist_yaw_0091_collision_geometric.obj"/>
+          <mesh filename="package://dvrk_model/meshes/instruments/wrist_yaw/0091/collision_hulls/wrist_yaw_0091_convex_hull_00.obj"/>
         </geometry>
         <material name="collision_red"><color rgba="1.0 0.0 0.0 1.0"/></material>
